File: schematics/ADAHRS-accelerometer-LRU-v1_00.kicad_sch (KiCad schematic)
At the start: 9 parts

Commit message: Add files via upload
Connections:
- net ADXL_CS renamed MCU CS
- net ADXL_MISO renamed MCU MISO
- net ADXL_MOSI renamed MCU MOSI
- net ADXL_SCLK renamed MCU SCLK
Changed lines of the file:
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@@
 	(title_block
 		(title "adahrs-accel-v1_00")
-		(rev "A")
-		(comment 1 "Will be integrated with custom SBC")
+		(rev "B")
+		(comment 1 "I need to integrate a crystal osc")
 	)
 	(junction
@@
 		)
 	)
-	(global_label "ADXL_CS"
+	(global_label "MCU CS"
 		(shape input)
 		(at 172.72 132.08 0)
@@
 		)
 		(property "Intersheetrefs" "${INTERSHEET_REFS}"
-			(at 183.7485 132.08 0)
+			(at 183.2042 132.08 0)
 			(effects
 				(font
@@
 		)
 	)
-	(global_label "ADXL_SCLK"
+	(global_label "MCU SCLK"
 		(shape input)
 		(at 172.72 127 0)
@@
 		)
 		(property "Intersheetrefs" "${INTERSHEET_REFS}"
-			(at 186.0466 127 0)
+			(at 185.5023 127 0)
 			(effects
 				(font
@@
 		)
 	)
-	(global_label "ADXL_MOSI"
+	(global_label "MCU MOSI"
 		(shape input)
 		(at 172.72 121.92 0)
@@
 		)
 		(property "Intersheetrefs" "${INTERSHEET_REFS}"
-			(at 185.8652 121.92 0)
+			(at 185.3209 121.92 0)
 			(effects
 				(font
@@
 		)
 	)
-	(global_label "ADXL_MISO"
+	(global_label "MCU MISO"
 		(shape input)
 		(at 173.355 116.84 0)
@@
 		)
 		(property "Intersheetrefs" "${INTERSHEET_REFS}"
-			(at 186.5002 116.84 0)
+			(at 185.9559 116.84 0)
 			(effects
 				(font
