File: schematics/ADAHRS-barometer.kicad_sch (KiCad schematic)
At the start: 5 parts

Commit message: Renamed and fixed labels v1.01
Parts:
- R1, R3, R4: value 10k -> 10kΩ
Connections:
- net MCU SPI MISO renamed MCU SPI MISO BAROMETER
- net MCU SPI MOSI renamed MCU SPI MOSI BAROMETER
- net MCU SPI SCLK renamed MCU SPI SCLK BAROMETER
Changed lines of the file:
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@@
 		(title "Barometer")
 		(date "09/13/26")
-		(rev "-")
+		(rev "A")
 		(comment 1 "/SSA Has weak internal pullups; for noise immunity 10K-47K pull-up to Vs is recommended")
 		(comment 2 "EOC connect to the MCU GPIO interrupt input to give a positive 5 microfared when finished")
@@
 		)
 	)
-	(global_label "MCU SPI SCLK"
+	(global_label "MCU SPI SCLK BAROMETER"
 		(shape input)
 		(at 164.465 85.725 0)
@@
 		)
 		(property "Intersheetrefs" "${INTERSHEET_REFS}"
-			(at 181.2992 85.725 0)
+			(at 193.2129 85.725 0)
 			(effects
 				(font
@@
 		)
 	)
-	(global_label "MCU SPI MISO"
+	(global_label "MCU SPI MISO BAROMETER"
 		(shape input)
 		(at 108.585 86.995 180)
@@
 		)
 		(property "Intersheetrefs" "${INTERSHEET_REFS}"
-			(at 91.9322 86.995 0)
+			(at 80.0185 86.995 0)
 			(effects
 				(font
@@
 		)
 	)
-	(global_label "MCU SPI MOSI"
+	(global_label "MCU SPI MOSI BAROMETER"
 		(shape input)
 		(at 164.465 89.535 0)
@@
 		)
 		(property "Intersheetrefs" "${INTERSHEET_REFS}"
-			(at 181.1178 89.535 0)
+			(at 193.0315 89.535 0)
 			(effects
 				(font
@@
 			)
 		)
-		(property "Value" "10k"
+		(property "Value" "10kΩ"
 			(at 198.755 88.265 0)
 			(effects
@@
 			)
 		)
-		(property "Value" "10k"
+		(property "Value" "10kΩ"
 			(at 116.84 103.505 90)
 			(effects
@@
 		(dnp no)
 		(property "Reference" "R4"
-			(at 73.025 83.82 0)
-			(effects
-				(font
-					(size 1.27 1.27)
-				)
-			)
-		)
-		(property "Value" "10k"
-			(at 73.025 86.36 0)
-			(effects
-				(font
+			(at 73.66 86.36 0)
+			(effects
+				(font
+					(size 1.27 1.27)
+				)
+			)
+		)
+		(property "Value" "10kΩ"
+			(at 73.66 88.9 0)
+			(effects
+				(font
