File: schematics/ADAHRS-accelerometer.kicad_sch (KiCad schematic)
At the start: 9 parts

Commit message: renamed global leabels accel v1.04
I renamed the global labels.
Connections:
- net MCU GPIO 0 DRDY renamed MCU GPIO DRDY accel
- net MCU GPIO 1 INT1 renamed MCU GPIO 0 INT1
- net MCU GPIO 2 INT2 renamed MCU GPIO 1 INT2
Changed lines of the file:
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@@
 		(title "accelerometer")
 		(date "08/31/26")
-		(rev "C")
-		(comment 1 "I need to integrate a crystal osc")
+		(rev "D")
 	)
 	(junction
@@
 	(wire
 		(pts
-			(xy 99.695 92.71) (xy 143.51 92.71)
+			(xy 95.25 92.71) (xy 143.51 92.71)
 		)
 		(stroke
@@
 	(wire
 		(pts
-			(xy 99.695 92.71) (xy 99.695 116.84)
+			(xy 95.25 92.71) (xy 95.25 116.84)
 		)
 		(stroke
@@
 	(wire
 		(pts
-			(xy 99.695 116.84) (xy 135.255 116.84)
+			(xy 95.25 116.84) (xy 135.255 116.84)
 		)
 		(stroke
@@
 		)
 	)
-	(global_label "MCU GPIO 2 INT2"
+	(global_label "MCU GPIO 1 INT2"
 		(shape input)
 		(at 120.015 113.03 180)
@@
 		)
 	)
-	(global_label "MCU GPIO 1 INT1"
+	(global_label "MCU GPIO 0 INT1"
 		(shape input)
 		(at 120.015 107.95 180)
@@
 		)
 	)
-	(global_label "MCU GPIO 0 DRDY"
+	(global_label "MCU GPIO DRDY accel"
 		(shape input)
 		(at 120.015 102.87 180)
@@
 		)
 		(property "Intersheetrefs" "${INTERSHEET_REFS}"
-			(at 99.4917 102.87 0)
+			(at 95.6212 102.87 0)
 			(effects
 				(font
@@
 		(dnp no)
 		(property "Reference" "C7"
-			(at 95.885 114.3 90)
+			(at 99.06 123.19 90)
 			(effects
 				(font
@@
 		)
 		(property "Value" "0.1uF"
-			(at 95.885 116.84 90)
-			(effects
-				(font
+			(at 99.06 125.73 90)
+			(effects
+				(font
