File: schematics/ADAHRS-magnetometer-LRU.kicad_sch (KiCad schematic)
At the start: 46 parts, among them Q1 2N2222, Q2 IRF7171M, Q3 Q2 - 2N2907, Q4 2N2222, Q5 IRF7171M, U1 OPA365-EP, U3 OPA365-EP, Y1 32.768 kHz Crystal

Commit message: changes to external supply
Connections:
- net +3.3v from MCU renamed +3v3
- net MCU GND renamed MCU DGND
- net MCU GPIO/START renamed MCU GPIO/rSTART
- net MCU GPIO/interupt input renamed MCU GPIO/DRDY
- net MCU SPI MISO renamed MCU SPI MISO/DOUT
- net MCU SPI MOSI renamed MCU SPI MOSI/rDIN
- net MCU SPI chip-select renamed MCU SPI/CS
Changed lines of the file:
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@@
 		(title "magnetic header")
 		(date "2026-08-31")
-		(rev "-")
+		(rev "6")
 		(comment 1 "Will be a daughterboard due to the need of distance from other magnetic field interference.\n")
 		(comment 2 "The output of each 2kΩ needs an RFI filter")
+		(comment 3 "Check the CLKSEL and RESET on the ADC connected to the 3.3 from MCU")
 	)
 	(junction
@@
 		)
 	)
-	(global_label "MCU GND"
+	(global_label "MCU DGND"
 		(shape input)
 		(at 257.175 202.565 180)
@@
 		)
 		(property "Intersheetrefs" "${INTERSHEET_REFS}"
-			(at 245.2998 202.565 0)
+			(at 244.0298 202.565 0)
 			(effects
 				(font
@@
 		)
 	)
-	(global_label "+3.3v from MCU"
-		(shape input)
-		(at 351.79 216.535 0)
-		(fields_autoplaced yes)
-		(effects
-			(font
-				(size 1.27 1.27)
-			)
-			(justify left)
-		)
-		(property "Intersheetrefs" "${INTERSHEET_REFS}"
-			(at 370.6803 216.535 0)
-			(effects
-				(font
-					(size 1.27 1.27)
-				)
-				(justify left)
-				(hide yes)
-			)
-		)
-	)
-	(global_label "MCU SPI MISO"
+	(global_label "MCU SPI MISO{slash}DOUT"
 		(shape input)
 		(at 257.175 226.695 180)
@@
 		)
 		(property "Intersheetrefs" "${INTERSHEET_REFS}"
-			(at 240.5222 226.695 0)
+			(at 234.2931 226.695 0)
 			(effects
 				(font
@@
 		)
 	)
-	(global_label "MCU SPI MOSI"
+	(global_label "MCU SPI MOSI{slash}rDIN"
 		(shape input)
 		(at 257.175 231.14 180)
@@
 		)
 		(property "Intersheetrefs" "${INTERSHEET_REFS}"
-			(at 240.5222 231.14 0)
+			(at 235.2002 231.14 0)
 			(effects
 				(font
@@
 		)
 	)
-	(global_label "MCU GPIO{slash}interupt input"
+	(global_label "MCU GPIO{slash}DRDY"
 		(shape input)
 		(at 257.175 217.805 180)
@@
 		)
 		(property "Intersheetrefs" "${INTERSHEET_REFS}"
-			(at 230.2414 217.805 0)
+			(at 238.4659 217.805 0)
 			(effects
 				(font
@@
 		)
 	)
-	(global_label "+3.3v from MCU"
-		(shape input)
-		(at 239.395 206.375 180)
-		(fields_autoplaced yes)
-		(effects
-			(font
-				(size 1.27 1.27)
-			)
-			(justify right)
-		)
-		(property "Intersheetrefs" "${INTERSHEET_REFS}"
-			(at 220.5047 206.375 0)
-			(effects
-				(font
-					(size 1.27 1.27)
-				)
-				(justify right)
-				(hide yes)
-			)
-		)
-	)
-	(global_label "MCU GPIO{slash}START"
+	(global_label "MCU GPIO{slash}rSTART"
 		(shape input)
 		(at 257.175 213.995 180)
@@
 		)
 		(property "Intersheetrefs" "${INTERSHEET_REFS}"
-			(at 237.8612 213.995 0)
+			(at 237.075 213.995 0)
 			(effects
 				(font
@@
 		)
 	)
-	(global_label "MCU SPI chip-select"
+	(global_label "MCU SPI{slash}CS"
 		(shape input)
 		(at 257.175 210.185 180)
@@
 		)
 		(property "Intersheetrefs" "${INTERSHEET_REFS}"
-			(at 233.8698 210.185 0)
+			(at 242.276 210.185 0)
 			(effects
 				(font
@@
 	)
 	(symbol
+		(lib_id "power:+5V")
+		(at 351.79 216.535 270)
+		(unit 1)
+		(exclude_from_sim no)
+		(in_bom yes)
+		(on_board yes)
+		(dnp no)
+		(property "Reference" "#PWR037"
+			(at 347.98 216.535 0)
+			(effects
+				(font
+					(size 1.27 1.27)
+				)
+				(hide yes)
+			)
+		)
+		(property "Value" "+3v3"
+			(at 351.79 217.805 90)
+			(effects
+				(font
+					(size 1.27 1.27)
+				)
+				(justify left)
+			)
+		)
+		(property "Footprint" ""
+			(at 351.79 216.535 0)
+			(effects
+				(font
+					(size 1.27 1.27)
+				)
+				(hide yes)
+			)
+		)
+		(property "Datasheet" ""
+			(at 351.79 216.535 0)
+			(effects
+				(font
+					(size 1.27 1.27)
+				)
+				(hide yes)
+			)
+		)
+		(property "Description" "Power symbol creates a global label with name \"+5V\""
+			(at 351.79 216.535 0)
+			(effects
+				(font
+					(size 1.27 1.27)
+				)
+				(hide yes)
+			)
+		)
+		(pin "1"
+		)
+		(instances
+			(project "ADAHRS-magnetometer-LRU"
+				(path "/e09c11d5-dbc8-40db-913b-60a97a341fc2"
+					(reference "#PWR037")
+					(unit 1)
+				)
+			)
+		)
+	)
+	(symbol
 		(lib_id "power:GND")
 		(at 330.2 109.22 180)
@@
 					(unit 1)
 				)
+			)
+		)
+	)
+	(symbol
+		(lib_id "power:+5V")
+		(at 239.395 206.375 90)
+		(unit 1)
+		(exclude_from_sim no)
+		(in_bom yes)
+		(on_board yes)
+		(dnp no)
+		(property "Reference" "#PWR038"
+			(at 243.205 206.375 0)
+			(effects
+				(font
+					(size 1.27 1.27)
+				)
+				(hide yes)
+			)
+		)
+		(property "Value" "+3v3"
+			(at 238.76 208.28 90)
+			(effects
+				(font
+					(size 1.27 1.27)
+				)
+				(justify left)
+			)
+		)
+		(property "Footprint" ""
+			(at 239.395 206.375 0)
+			(effects
+				(font
+					(size 1.27 1.27)
+				)
+				(hide yes)
+			)
+		)
+		(property "Datasheet" ""
+			(at 239.395 206.375 0)
+			(effects
+				(font
+					(size 1.27 1.27)
+				)
+				(hide yes)
+			)
+		)
+		(property "Description" "Power symbol creates a global label with name \"+5V\""
+			(at 239.395 206.375 0)
+			(effects
+				(font
+					(size 1.27 1.27)
+				)
+				(hide yes)
+			)
+		)
+		(pin "1"
+		)
+		(instances
+			(project "ADAHRS-magnetometer-LRU"
+				(path "/e09c11d5-dbc8-40db-913b-60a97a341fc2"
+					(reference "#PWR038")
+					(unit 1)
+				)

Commit message: fixed pullup labels v1.07
I need to check all pull ups if I forgot to add the symbol ohms.
Parts:
- R18, R19: value 10k (pull-up) -> 10kΩ
Connections:
- net MCU DGND is gone; now on net +18v: U-ADS1258MRTCTEP.29 (DGND)
- net AIN6: now reaches U-ADS1258MRTCTEP.46 (AIN6)
- net MCU SPI/CS renamed MCU all analog SPI/CS

Commit message: Renamed global label magnetometer v1.07
I messed up the version on the last upload for magnetometer. Additionally, I added unconnected labels on the offset pins. I knew I wanted the ADC on the main board and the magnetometer needs to be at least 0.1 meters away from components that causes high electromagnetic interferences such as inductors. I made the AIN pins become global labels and added a simple RFI filter which specifically is a first-order RC low-pass filter. High frequencies are more likely to be muffled. The AIN pins will most likely need to be connected through JST or a molex style connector if I am doing a daughterboard of the magnetometer circuits. I could still have the magnetometer on the main PCB if the high electromagnetic components will be somewhat close to my design target of 0.1 meter. It is better for now to hold the AIN as global labels until I finish the schematic capture and start designing rough drafts on paper of how I want the LRU PCBs to be designed.
Parts:
- added C17, C19, C20: 1nF, symbol Device:C
- added C18: 2.2nF, symbol Device:C
- added R21, R23: 100Ω, symbol Device:R
- added R22: 47kΩ, symbol Device:R
- R16: value 47kΩ -> 100Ω
Connections:
- net +18v: now also C17.2, C19.2, C20.2
- net +3v3: no longer R18.1, R19.1
- net AIN6: now also R23.1; no longer U-ADS1258MRTCTEP.46 (AIN6)
- net AIN3: now reaches U-ADS1258MRTCTEP.1 (AIN3), U-HMC1002.12 (OUT-_B)
- net AIN2: now reaches R10.2, U-ADS1258MRTCTEP.2 (AIN2)
- net AIN1: now reaches R9.2, U-ADS1258MRTCTEP.3 (AIN1)
- net AIN0: now reaches R8.2, U-ADS1258MRTCTEP.4 (AIN0)
- net at U-ADS1258MRTCTEP.41 (ADCINN): now also C18.2, R22.1; no longer R15.2
- net at U-ADS1258MRTCTEP.42 (ADCINP): now also R15.1, C18.1; no longer R16.2
- net at U-ADS1258MRTCTEP.47 (AIN5): now also C19.1, R21.2; no longer R12.1
- net at U-ADS1258MRTCTEP.48 (AIN4): now also R16.2, C17.1; no longer R11.1
- net at R14.2, R17.1, U3.4 (-): now also R22.2; no longer R15.1
- net at R13.2, R17.2, U1.4 (-): now also R15.2; no longer R16.1
- new net: C20.1, R23.2, U-ADS1258MRTCTEP.46 (AIN6)
- new net +3V3: R18.1, R19.1
- new net AIN4: R11.1, R16.1
- new net AIN5: R12.1, R21.1
- no-connect marks 2 -> 7
Other:
- moved on the sheet: C5, C6, R10, R13, R14, R17, R8, R9, U1, U3
